File: 07-clifford1one/sesion-14b/archivos/fps555/fps555.kicad_sch (KiCad schematic)
At the start: 29 parts, among them M4 Motor_DC, Q1 IRLZ44N, Q2 IRLZ44N, SW1 SW_SPST, SW2 SW_SPST, SW3 SW_SPST, SW4 SW_SPST, U1 555, U3 555

Commit message: Update fps555.kicad_sch
Parts:
- added U2: L293D, Package_DIP:DIP-16_W7.62mm, symbol Driver_Motor:L293D
Changed lines of the file:
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@@
+	)
+	(symbol
+		(lib_id "Driver_Motor:L293D")
+		(at 194.31 54.61 0)
+		(unit 1)
+		(exclude_from_sim no)
+		(in_bom yes)
+		(on_board yes)
+		(dnp no)
+		(fields_autoplaced yes)
+		(property "Reference" "U2"
+			(at 198.9933 26.67 0)
+			(effects
+				(font
+					(size 1.27 1.27)
+				)
+				(justify left)
+			)
+		)
+		(property "Value" "L293D"
+			(at 198.9933 29.21 0)
+			(effects
+				(font
+					(size 1.27 1.27)
+				)
+				(justify left)
+			)
+		)
+		(property "Footprint" "Package_DIP:DIP-16_W7.62mm"
+			(at 200.66 73.66 0)
+			(effects
+				(font
+					(size 1.27 1.27)
+				)
+				(justify left)
+				(hide yes)
+			)
+		)
+		(property "Datasheet" "http://www.ti.com/lit/ds/symlink/l293.pdf"
+			(at 186.69 36.83 0)
+			(effects
+				(font
+					(size 1.27 1.27)
+				)
+				(hide yes)
+			)
+		)
+		(property "Description" "Quadruple Half-H Drivers"
+			(at 194.31 54.61 0)
+			(effects
+				(font
+					(size 1.27 1.27)
+				)
+				(hide yes)
+			)
+		)
+		(pin "1"
+		)
+		(pin "3"
+		)
+		(pin "15"
+		)
+		(pin "9"
+		)
+		(pin "12"
+		)
+		(pin "7"
+		)
+		(pin "2"
+		)
+		(pin "11"
+		)
+		(pin "14"
+		)
+		(pin "8"
+		)
+		(pin "4"
+		)
+		(pin "16"
+		)
+		(pin "13"
+		)
+		(pin "5"
+		)
+		(pin "10"
+		)
+		(pin "6"
+		)
+		(instances
+			(project ""
+				(path "/17d5fafb-d426-46d5-861d-7151424b81f3"
+					(reference "U2")
+					(unit 1)
+				)
+			)
+		)
 	)
 	(symbol
