File: 07-clifford1one/sesion-15a/archivos/fps555-v3.kicad_sch (KiCad schematic)
At the start: 18 parts, among them M1 Motorreductor, SW3 SW_SPDT_MSM, U1 555, U2 L293D

Commit message: cambios sch
Connections:
- net at U2.1 (EN1,2): now also R3.2, R4.1, SW3.2 (3)
Changed lines of the file:
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@@
+	)
+	(junction
+		(at 105.41 62.23)
+		(diameter 0)
+		(color 0 0 0 0)
 	)
 	(junction
@@
 	)
 	(junction
+		(at 121.92 62.23)
+		(diameter 0)
+		(color 0 0 0 0)
+	)
+	(junction
 		(at 208.28 39.37)
 		(diameter 0)
@@
 	(wire
 		(pts
+			(xy 132.08 52.07) (xy 121.92 52.07)
+		)
+		(stroke
+			(width 0)
+			(type default)
+		)
+	)
+	(wire
+		(pts
 			(xy 31.75 73.66) (xy 31.75 72.39)
 		)
@@
 	(wire
 		(pts
+			(xy 121.92 52.07) (xy 121.92 62.23)
+		)
+		(stroke
+			(width 0)
+			(type default)
+		)
+	)
+	(wire
+		(pts
 			(xy 175.26 49.53) (xy 195.58 49.53)
 		)
@@
 	(wire
 		(pts
+			(xy 105.41 62.23) (xy 121.92 62.23)
+		)
+		(stroke
+			(width 0)
+			(type default)
+		)
+	)
+	(wire
+		(pts
 			(xy 49.53 67.31) (xy 49.53 73.66)
 		)
@@
 		)
 		(stroke
+			(width 0)
+			(type default)
+		)
+	)
+	(wire
+		(pts
+			(xy 121.92 62.23) (xy 146.05 62.23)
+		)
+		(stroke
