File: 07-clifford1one/sesion-15a/archivos/fps555-v5.kicad_sch (KiCad schematic)
At the start: 21 parts, among them M1 Motorreductor, U1 555, U2 L293D

Commit message: archivos nuevo sch
Connections:
- net GND: no longer U2.12 (GND), U2.13 (GND)
- no-connect marks 5 -> 7
Changed lines of the file:
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@@
 	)
 	(junction
-		(at 148.59 87.63)
-		(diameter 0)
-		(color 0 0 0 0)
-	)
-	(junction
 		(at 177.8 76.2)
 		(diameter 0)
@@
 	)
 	(no_connect
+		(at 149.86 87.63)
+	)
+	(no_connect
 		(at 132.08 72.39)
 	)
@@
 		(at 132.08 77.47)
 	)
+	(no_connect
+		(at 147.32 87.63)
+	)
 	(wire
 		(pts
@@
 	(wire
 		(pts
-			(xy 147.32 87.63) (xy 148.59 87.63)
-		)
-		(stroke
-			(width 0)
-			(type default)
-		)
-	)
-	(wire
-		(pts
 			(xy 109.22 54.61) (xy 109.22 50.8)
 		)
@@
 	(wire
 		(pts
-			(xy 148.59 87.63) (xy 149.86 87.63)
-		)
-		(stroke
-			(width 0)
-			(type default)
-		)
-	)
-	(wire
-		(pts
 			(xy 104.14 62.23) (xy 105.41 62.23)
 		)
@@
 	)
 	(symbol
-		(lib_id "power:GND")
-		(at 148.59 87.63 0)
-		(unit 1)
-		(exclude_from_sim no)
-		(in_bom yes)
-		(on_board yes)
-		(dnp no)
-		(fields_autoplaced yes)
-		(property "Reference" "#PWR020"
-			(at 148.59 93.98 0)
-			(effects
-				(font
-					(size 1.27 1.27)
-				)
-				(hide yes)
-			)
-		)
-		(property "Value" "GND"
-			(at 148.59 92.71 0)
-			(effects
-				(font
-					(size 1.27 1.27)
-				)
-			)
-		)
-		(property "Footprint" ""
-			(at 148.59 87.63 0)
-			(effects
-				(font
-					(size 1.27 1.27)
-				)
-				(hide yes)
-			)
-		)
-		(property "Datasheet" ""
-			(at 148.59 87.63 0)
-			(effects
-				(font
-					(size 1.27 1.27)
-				)
-				(hide yes)
-			)
-		)
-		(property "Description" "Power symbol creates a global label with name \"GND\" , ground"
-			(at 148.59 87.63 0)
-			(effects
-				(font
-					(size 1.27 1.27)
-				)
-				(hide yes)
-			)
-		)
-		(pin "1"
-		)
-		(instances
-			(project "fps555-v4"
-				(path "/17d5fafb-d426-46d5-861d-7151424b81f3"
-					(reference "#PWR020")
-					(unit 1)
-				)
-			)
-		)
-	)
-	(symbol
 		(lib_id "Device:R_US")
 		(at 128.27 45.72 180)
@@
 		)
 		(property "Value" "100k"
-			(at 95.504 50.546 0)
+			(at 94.361 50.165 0)
 			(effects
 				(font
