File: 07-clifford1one/sesion-15a/archivos/fps555-v5.2.kicad_pcb (KiCad board)
At the start: 2 copper layers, 212 x 110 mm, 21 parts, among them M1 Motorreductor, U1 555, U2 L293D, U3 mst303

Commit message: cambios kicad
Parts:
- added D8: 4007, Diode_THT:D_A-405_P10.16mm_Horizontal, F.Cu at (31.8, 82.8)
- added J1: Screw_Terminal_01x02, TerminalBlock:TerminalBlock_MaiXu_MX126-5.0-02P_1x02_P5.00mm, F.Cu at (34.0, 62.0)
- R2: value 1k -> 10k
- moved D2 18.2 mm to (47.0, 60.8)
- moved D3 18.2 mm to (41.0, 71.0)
- moved C2 18.1 mm to (59.5, 76.0)
- moved R5 17.1 mm to (122.0, 80.1)
- moved R6 17.1 mm to (117.0, 80.1)
- moved R7 17.1 mm to (112.0, 70.0)
- moved U3 17.0 mm to (134.0, 75.0)
- moved M1 15.0 mm to (131.0, 65.0)
- moved R2 11.5 mm to (63.4, 68.4), turned to 180 degrees
- moved C1 11.4 mm to (63.0, 81.0)
- moved D1 9.73 mm to (117.0, 59.0)
- moved U1 8.85 mm to (45.9, 82.0)
- moved R1 6.26 mm to (52.9, 56.5)
- moved R3 6.26 mm to (53.0, 60.5)
- moved R4 6.26 mm to (52.8, 64.5)
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Other:
- board size 212 x 110 mm -> 109.8 x 48 mm
