File: 07-clifford1one/sesion-15a/archivos/fps555-v5.2.kicad_pcb (KiCad board)
At the start: 2 copper layers, 100 x 50 mm, 23 parts, among them J1 Batería 9v, M1 Motorreductor, U1 555, U2 L293D, U3 mst303

Commit message: cambios pcb
Routing:
- net GND: track 213.9 -> 174.7 mm
- net Net-(U2-1A): track 83.6 -> 73.5 mm
- added copper zone on B.Cu, net (none)
Changed lines of the file:
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@@
-	(gr_poly
-		(pts
-			(xy 89.403922 51.977335) (xy 89.366019 52.002046) (xy 89.118329 52.09752) (xy 88.828787 52.205231)
-			(xy 88.49342 52.324814) (xy 87.161918 52.941689) (xy 85.781959 53.879654) (xy 84.543291 54.987222)
-			(xy 83.639751 56.116618) (xy 83.306184 56.661884) (xy 83.089326 57.093805) (xy 82.935435 57.523925)
-			(xy 82.803255 58.056838) (xy 82.737404 58.336789) (xy 82.675636 58.507708) (xy 82.611943 58.597667)
-			(xy 82.541781 58.615779) (xy 82.079033 58.516709) (xy 81.290759 58.408275) (xy 80.480173 58.320717)
-			(xy 79.891243 58.28893) (xy 79.105968 58.298284) (xy 78.062212 58.351902) (xy 76.99387 58.424108)
-			(xy 76.807476 58.484082) (xy 76.685491 58.53302) (xy 76.086367 58.659197) (xy 75.511595 58.772191)
-			(xy 75.153323 58.82556) (xy 75.061324 58.825083) (xy 75.006746 58.797016) (xy 74.980723 58.738604)
-			(xy 74.98132 58.639047) (xy 74.978923 58.550649) (xy 74.954571 58.457452) (xy 74.913311 58.37337)
-			(xy 74.860414 58.31292) (xy 74.805961 58.25139) (xy 74.760021 58.163713) (xy 74.728717 58.065235)
-			(xy 74.718159 57.97072) (xy 74.711083 57.880519) (xy 74.689854 57.794881) (xy 74.658669 57.725432)
-			(xy 74.621486 57.68681) (xy 74.584423 57.650465) (xy 74.553238 57.589413) (xy 74.532009 57.515528)
-			(xy 74.524808 57.439366) (xy 74.517737 57.36752) (xy 74.496383 57.306826) (xy 74.465079 57.265926)
-			(xy 74.428135 57.251654) (xy 74.391072 57.232461) (xy 74.359887 57.172727) (xy 74.338539 57.085888)
-			(xy 74.331462 56.982976) (xy 74.317787 56.865671) (xy 74.277367 56.750404) (xy 74.215355 56.649531)
-			(xy 74.137992 56.574806) (xy 74.06411 56.512195) (xy 74.001496 56.439628) (xy 73.958192 56.368023)
-			(xy 73.944641 56.310089) (xy 73.920293 56.234881) (xy 73.776477 56.044651) (xy 73.591525 55.822156)
-			(xy 73.372265 55.582147) (xy 73.129499 55.321507) (xy 72.87342 55.036879) (xy 72.640842 54.77012)
-			(xy 72.477841 54.572211) (xy 72.097136 54.160565) (xy 71.665218 53.822443) (xy 71.028794 53.448454)
-			(xy 69.884882 52.867202) (xy 68.290582 52.078688) (xy 72.592148 52.028792) (xy 77.54525 51.984292)
-			(xy 83.300067 51.957066) (xy 89.387845 51.938833)
-		)
-		(stroke
-			(width 0.086359)
-			(type solid)
-		)
-		(fill no)
-		(layer "F.SilkS")
-	)
 	(gr_poly
 		(pts
@@
 	)
 	(segment
-		(start 74.938169 62.59617)
-		(end 53.576711 62.59617)
-		(width 0.2)
-		(layer "F.Cu")
-		(net 2)
-	)
-	(segment
 		(start 100 71.760568)
 		(end 93.421587 71.760568)
@@
 	)
 	(segment
-		(start 78.327679 59.20666)
-		(end 74.938169 62.59617)
-		(width 0.2)
-		(layer "F.Cu")
-		(net 2)
-	)
-	(segment
-		(start 53.576711 63.076711)
-		(end 53.576711 62.59617)
-		(width 0.2)
-		(layer "F.Cu")
-		(net 2)
-	)
-	(segment
 		(start 100.160018 79.032762)
 		(end 100.160018 75.240018)
@@
 	)
 	(segment
-		(start 62.5 72)
-		(end 53.576711 63.076711)
-		(width 0.2)
-		(layer "F.Cu")
-		(net 2)
-	)
-	(segment
 		(start 65 74.5)
 		(end 62.5 72)
@@
 	)
 	(segment
+		(start 54.203208 62.767498)
+		(end 54.203208 59.171328)
+		(width 0.2)
+		(layer "F.Cu")
+		(net 10)
+	)
+	(segment
 		(start 54.203208 75.876792)
 		(end 54.203208 62.767498)
@@
 	)
 	(segment
-		(start 54.203208 59.171328)
-		(end 54.203208 62.767498)
-		(width 0.2)
-		(layer "B.Cu")
-		(net 10)
-	)
-	(segment
 		(start 56.325046 50.48566)
 		(end 44.043208 62.767498)
@@
 	)
 	(segment
-		(start 125.35003 71.760568)
-		(end 126.263446 72.673984)
-		(width 0.2)
-		(layer "F.Cu")
-		(net 13)
-	)
-	(segment
 		(start 87.048679 50.48566)
 		(end 117.42413 50.48566)
@@
 	(segment
 		(start 124.886667 65.037935)
-		(end 118.164034 71.760568)
+		(end 121.712301 68.212301)
 		(width 0.2)
 		(layer "F.Cu")
@@
 	)
 	(segment
+		(start 121.712301 68.212301)
+		(end 118.164034 71.760568)
+		(width 0.2)
+		(layer "F.Cu")
+		(net 13)
+	)
+	(segment
 		(start 117.42413 50.48566)
 		(end 124.886667 57.948197)
@@
 	)
 	(segment
-		(start 110.16 71.760568)
-		(end 125.35003 71.760568)
+		(start 126.263446 72.673984)
+		(end 126.173984 72.673984)
 		(width 0.2)
 		(layer "F.Cu")
@@
 	)
 	(segment
+		(start 126.173984 72.673984)
+		(end 121.712301 68.212301)
+		(width 0.2)
+		(layer "F.Cu")
+		(net 13)
+	)
+	(segment
 		(start 110.320018 79.032762)
 		(end 113.678796 75.673984)
@@
 		(net 21)
 	)
+	(zone
+		(net 0)
+		(net_name "")
+		(layer "B.Cu")
+		(hatch edge 0.5)
+		(connect_pads
+			(clearance 0.5)
+		)
+		(min_thickness 0.25)
+		(filled_areas_thickness no)
+		(fill yes
+			(thermal_gap 0.5)
+			(thermal_bridge_width 0.5)
+			(island_removal_mode 1)
+			(island_area_min 10)
+		)
+		(polygon
+			(pts
+				(xy 25 37.5) (xy 27 100.5) (xy 139.5 100.5) (xy 139.5 39)
+			)
+		)
+	)
 	(group ""
-		(members "3e8d539b-d437-4997-82b9-79e873132376" "e73c6a3b-8d21-4230-85cf-ac5daf9a33af")
+		(members "e73c6a3b-8d21-4230-85cf-ac5daf9a33af")
 	)
 	(embedded_fonts no)

Commit message: cambios pcb
Parts:
- U3: footprint Connector_PinHeader_1.00mm:PinHeader_1x05_P1.00mm_Vertical -> Connector_PinHeader_2.54mm:PinHeader_1x05_P2.54mm_Vertical
- moved U3 6.21 mm to (125.5, 78.8)
- moved RV1 2.01 mm to (74.6, 71.0)
- moved D8 1.87 mm to (34.8, 85.2)
- moved R4 1.42 mm to (44.0, 66.8)
- moved R2 0.91 mm to (44.0, 55.0)
- moved R5 0.51 mm to (100.0, 75.5)
- moved C2 0.45 mm to (67.0, 72.0)
- moved R7 0.16 mm to (100.0, 79.0)
Routing:
- net GND: track 174.7 -> 190.7 mm
- net Net-(U2-1A): track 73.5 -> 79.3 mm
- net Net-(D2-K): track 25.6 -> 30.5 mm
- net Net-(U2-2A): track 63.5 -> 66.9 mm
- net VCC: track 153.6 -> 156.3 mm
- net Net-(U1-R): track 75.5 -> 77.9 mm
- net Net-(U1-THR): track 55.3 -> 56.8 mm
- net +9V: track 9.64 -> 11.1 mm
- net Net-(D3-K): track 23.3 -> 22.1 mm
- net Net-(U2-EN1,2): track 54.6 -> 54.0 mm
- removed copper zone on B.Cu, net (none)
