File: 07-clifford1one/sesion-15a/archivos/fps555-v11cm.kicad_pcb (KiCad board)
At the start: 2 copper layers, 100 x 55 mm, 23 parts, among them J1 Batería 9v, M1 Motorreductor, U1 555, U2 L293D, U3 mst303

Commit message: CAMBIOS KICAD
Parts:
- J1: value Batería 9v -> Screw_Terminal_01x02
- moved U1 10.9 mm to (45.9, 82.0), turned to 90 degrees
- moved R5 9.41 mm to (122.0, 80.1)
- moved R6 9.41 mm to (117.0, 80.1)
- moved R7 9.41 mm to (112.0, 70.0)
- moved U3 8.08 mm to (134.0, 75.0)
- moved M1 7.93 mm to (131.0, 65.0)
- moved D3 6.34 mm to (41.0, 71.0)
- moved D5 6.06 mm to (96.9, 67.0)
- moved D4 6.06 mm to (107.1, 71.0)
- moved D1 6.02 mm to (117.0, 59.0)
- moved D2 5.83 mm to (47.0, 60.8)
- moved C1 5.39 mm to (63.0, 81.0)
- moved C2 4.47 mm to (59.5, 76.0)
- moved D7 4.17 mm to (107.3, 61.0)
- moved D6 4.17 mm to (97.0, 57.0)
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Connections:
- D5 pad 1: VCC -> +5V
- D7 pad 1: VCC -> +5V
- R2 pad 1: VCC -> +5V
- U1 pad 8: VCC -> +5V
- U2 pad 16: VCC -> +5V
- U2 pad 8: VCC -> +5V
- U3 pad 2: VCC -> +5V
- U3 pad 5: VCC -> +5V
Other:
- board size 100 x 55 mm -> 109.8 x 48 mm
