File: 07-clifford1one/sesion-15a/archivos/fps555-vsilkGlass.kicad_pcb (KiCad board)
At the start: 2 copper layers, 100 x 50 mm, 23 parts, among them J1 Batería 9v, M1 Motorreductor, U1 555, U2 L293D, U3 mst303

Commit message: cambios >PCB
Parts:
- moved D1 75.1 mm to (37.5, 50.0)
Routing:
- net Net-(D1-A): track 76.3 -> 6.99 mm
- net GND: track 213.9 -> 219.1 mm
