File: 15-sz-mada/sesion-15a/kicad-proj02/kicad-proj02.kicad_pcb (KiCad board)
At the start: 2 copper layers, 35 parts, among them Q1 PN2222A, U1 555, U2 LM324, U3 4017, U4 555, U5 555

Commit message: kicad updated
Parts:
- removed D12: LED, LED_THT:LED_D5.0mm
- removed R13: 1k, Resistor_THT:R_Axial_DIN0207_L6.3mm_D2.5mm_P10.16mm_Horizontal
- added C1: 474, Capacitor_THT:C_Disc_D5.0mm_W2.5mm_P5.00mm, F.Cu at (105.2, 68.7)
- added C4: 474, Capacitor_THT:C_Disc_D5.0mm_W2.5mm_P5.00mm, F.Cu at (107.2, 87.7)
- added C7: C7, Capacitor_THT:C_Disc_D5.0mm_W2.5mm_P5.00mm, F.Cu at (227.8, 61.5)
- added MK1: Mic electret, Sensor_Audio:POM-2244P-C3310-2-R, F.Cu at (204.1, 72.0)
- added REF**: TerminalBlock_MaiXu_MX126-5.0-02P_1x02_P5.00mm, TerminalBlock:TerminalBlock_MaiXu_MX126-5.0-02P_1x02_P5.00mm, F.Cu at (92.8, 24.0)
- added RV1: 500k, Potentiometer_THT:Potentiometer_Piher_T-16H_Single_Horizontal, F.Cu at (79.8, 44.2)
- R10, R3, R8: value 1k -> 10k
- R12, R9: value 10k -> 1k
- R6: value 10k -> 100k
- R7: value 100k -> 1k
- moved R12 203.4 mm to (227.8, 55.8), turned to 90 degrees
- moved R11 192.3 mm to (216.8, 40.0)
- moved R10 185.1 mm to (209.6, 43.9), turned to 90 degrees
- moved C6 183.6 mm to (221.8, 64.5), turned to 180 degrees
- moved U5 180.9 mm to (213.1, 47.8)
- moved R9 179.9 mm to (204.3, 33.8), turned to -90 degrees
- moved C5 168.8 mm to (206.3, 62.0), turned to 180 degrees
- moved Q1 167.1 mm to (205.3, 54.5), turned to 90 degrees
- moved U2 81.7 mm to (86.5, 49.9)
- moved R8 81.7 mm to (212.6, 71.8), turned to 90 degrees
- moved U3 79.8 mm to (79.6, 81.5)
- moved U4 78.6 mm to (99.2, 74.4)
- moved R2 72.9 mm to (79.5, 72.2), turned to 90 degrees
- moved C3 63.1 mm to (93.0, 75.2), turned to 180 degrees
- moved R6 61.5 mm to (95.8, 88.3), turned to -90 degrees
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Connections:
- D1 pad 1: GND -> Net-(D1-K)
- D10 pad 1: Net-(D10-K) -> Net-(D1-K)
- D11 pad 1: Net-(D10-K) -> GND
- D2 pad 1: Net-(D10-K) -> Net-(D1-K)
- D3 pad 1: Net-(D10-K) -> Net-(D1-K)
- D4 pad 1: Net-(D10-K) -> Net-(D1-K)
- D5 pad 1: Net-(D10-K) -> Net-(D1-K)
- D6 pad 1: Net-(D10-K) -> Net-(D1-K)
- D7 pad 1: Net-(D10-K) -> Net-(D1-K)
- D8 pad 1: Net-(D10-K) -> Net-(D1-K)
- D9 pad 1: Net-(D10-K) -> Net-(D1-K)
- R11 pad 2: Net-(Q1-C) -> Net-(U5-DIS)
- R12 pad 1: +9V -> Net-(U5-Q)
- R12 pad 2: Net-(U5-DIS) -> Net-(D11-A)
- R3 pad 1: Net-(U1-TR) -> +9V
- R3 pad 2: Net-(D1-A) -> Net-(U1-DIS)
- R4 pad 2: Net-(U1-DIS) -> Net-(U4-DIS)
- R5 pad 1: +9V -> Net-(U4-DIS)
- R5 pad 2: Net-(U4-DIS) -> Net-(U4-THR)
- R6 pad 1: Net-(U4-DIS) -> Net-(U3-CKEN)
- R6 pad 2: Net-(U4-THR) -> GND
- R7 pad 1: Net-(U3-CKEN) -> Net-(D1-K)
- R8 pad 1: Net-(D10-K) -> +9V
- R8 pad 2: GND -> Net-(MK1-+)
- R9 pad 2: Net-(MK1-+) -> Net-(Q1-C)
- U3 pad 1: Net-(D10-A) -> Net-(D6-A)
- U3 pad 10: Net-(D6-A) -> Net-(D5-A)
- U3 pad 11: Net-(D9-A) -> Net-(D10-A)
- U3 pad 2: Net-(D7-A) -> Net-(D2-A)
- U3 pad 3: Net-(D3-A) -> Net-(D1-A)
- U3 pad 4: Net-(D5-A) -> Net-(D3-A)
- U3 pad 5: Net-(D2-A) -> Net-(D7-A)
- U3 pad 6: Net-(D11-A) -> Net-(D8-A)
- U3 pad 7: Net-(D8-A) -> Net-(D4-A)
- U3 pad 9: Net-(D4-A) -> Net-(D9-A)
Other:
- board outline added: 182.8 x 90 mm
