File: 15-sz-mada/sesion-15a/kicad-proj02/kicad-proj02.kicad_sch (KiCad schematic)
At the start: 40 parts, among them Q1 PN2222A, U1 555, U2 LM324, U3 4017, U4 555, U5 555

Commit message: kicad
Parts:
- C1, C4, C7: value 100n -> 474; footprint Capacitor_THT:C_Disc_D6.0mm_W2.5mm_P5.00mm -> (none)
- R4: value 220 -> 10k
- R5, R6: value 1k -> 10k
- R8: value 470 -> 1k
Other:
- note removed: "REVISAR HUELLA"
Changed lines of the file:
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@@
 		(title "Proyecto-02 - Grupo 05")
 	)
-	(text "Micrófono engañoso (no afecta ruleta)"
+	(text "AÑADIR\nHUELLA"
 		(exclude_from_sim no)
-		(at 91.948 112.776 0)
+		(at 125.73 167.132 0)
 		(effects
 			(font
 				(size 1.27 1.27)
 			)
+			(justify left)
 		)
 	)
-	(text "REVISAR\nHUELLA"
+	(text "Micrófono engañoso (no afecta ruleta)"
 		(exclude_from_sim no)
-		(at 78.74 154.178 0)
+		(at 91.948 112.776 0)
 		(effects
 			(font
 				(size 1.27 1.27)
 			)
-			(justify left)
 		)
 	)
@@
 		)
 	)
-	(text "REVISAR\nHUELLA"
-		(exclude_from_sim no)
-		(at 182.626 44.196 0)
-		(effects
-			(font
-				(size 1.27 1.27)
-			)
-			(justify right)
-		)
-	)
 	(text "AÑADIR\nHUELLA"
 		(exclude_from_sim no)
@@
 	(text "AÑADIR\nHUELLA"
 		(exclude_from_sim no)
-		(at 53.34 151.892 0)
+		(at 152.146 87.376 0)
 		(effects
 			(font
@@
 		)
 	)
-	(text "REVISAR\nHUELLA"
+	(text "AÑADIR\nHUELLA"
 		(exclude_from_sim no)
-		(at 58.674 70.358 0)
+		(at 108.966 87.884 0)
 		(effects
 			(font
 				(size 1.27 1.27)
 			)
+			(justify left)
 		)
 	)
-	(text "REVISAR\nHUELLA"
+	(text "AÑADIR\nHUELLA"
 		(exclude_from_sim no)
-		(at 36.576 42.926 0)
+		(at 53.34 151.892 0)
 		(effects
 			(font
 				(size 1.27 1.27)
 			)
-			(justify right)
+			(justify left)
 		)
 	)
@@
 			)
 		)
-		(property "Value" "100n"
+		(property "Value" "474"
 			(at 127 162.5599 0)
 			(effects
@@
 			)
 		)
-		(property "Footprint" "Capacitor_THT:C_Disc_D6.0mm_W2.5mm_P5.00mm"
+		(property "Footprint" ""
 			(at 124.1552 165.1 0)
 			(effects
@@
 			)
 		)
-		(property "Value" "100n"
+		(property "Value" "474"
 			(at 110.49 83.8199 0)
 			(effects
@@
 			)
 		)
-		(property "Footprint" "Capacitor_THT:C_Disc_D6.0mm_W2.5mm_P5.00mm"
+		(property "Footprint" ""
 			(at 107.6452 86.36 0)
 			(effects
@@
 			)
 		)
-		(property "Value" "100n"
+		(property "Value" "474"
 			(at 153.67 82.5499 0)
 			(effects
@@
 			)
 		)
-		(property "Footprint" "Capacitor_THT:C_Disc_D6.0mm_W2.5mm_P5.00mm"
+		(property "Footprint" ""
 			(at 150.8252 85.09 0)
 			(effects
@@
 			)
 		)
-		(property "Value" "220"
+		(property "Value" "10k"
 			(at 88.9 54.6099 0)
 			(effects
@@
 			)
 		)
-		(property "Value" "1k"
+		(property "Value" "10k"
 			(at 127 64.7699 0)
 			(effects
@@
 			)
 		)
-		(property "Value" "1k"
+		(property "Value" "10k"
 			(at 127 53.3399 0)
 			(effects
@@
 			)
 		)
-		(property "Value" "470"
+		(property "Value" "1k"
 			(at 193.294 91.694 90)
 			(effects

Commit message: kicad updated
Parts:
- removed D1: LED, LED_THT:LED_D5.0mm, symbol Device:LED
- removed R3: 1k, Resistor_THT:R_Axial_DIN0207_L6.3mm_D2.5mm_P10.16mm_Horizontal, symbol Device:R
- C1, C4, C7: footprint (none) -> Capacitor_THT:C_Disc_D5.0mm_W2.5mm_P5.00mm
- MK1: footprint (none) -> Sensor_Audio:POM-2244P-C3310-2-R
- RV1: footprint (none) -> Potentiometer_THT:Potentiometer_Piher_T-16H_Single_Horizontal
- renumbered D3 to D1, D9 to D10, D12 to D11, D7 to D2, D5 to D3, D8 to D4, D6 to D5, D10 to D6, D2 to D7, D11 to D8, D4 to D9, R11 to R10, R12 to R11, R13 to R12, R4 to R3, R5 to R4, R6 to R5, R7 to R6, R8 to R7, R9 to R8, R10 to R9
Other:
- note removed: "AÑADIR HUELLA"
- moved on the sheet: R1, R2, RV1, U2A
