File: 00-proyecto-02/grupo-05/kicad/proj02-g05.kicad_pcb (KiCad board)
At the start: 2 copper layers, 182.8 x 90 mm, 39 parts, among them Q1 PN2222A, U1 555, U2 LM324, U3 4017, U4 555, U5 555

Commit message: proyecto2
Parts:
- removed REF**: TerminalBlock_MaiXu_MX126-5.0-02P_1x02_P5.00mm, TerminalBlock:TerminalBlock_MaiXu_MX126-5.0-02P_1x02_P5.00mm
- C7: value C7 -> 474
- Q1: footprint Package_TO_SOT_THT:TO-92_Inline -> Package_TO_SOT_THT:TO-92_Inline_Wide
- moved D7 157.3 mm to (22.8, 38.8)
- moved D6 148.0 mm to (22.6, 50.2)
- moved D5 132.9 mm to (22.8, 61.8)
- moved R1 126.5 mm to (35.7, 81.0)
- moved D4 122.7 mm to (22.5, 72.9)
- moved D1 122.4 mm to (22.5, 110.2)
- moved D3 122.3 mm to (22.6, 85.5)
- moved D2 122.2 mm to (22.6, 97.5)
- moved R7 105.7 mm to (62.5, 108.8), turned to 90 degrees
- moved R10 104.3 mm to (105.5, 37.0), turned to -90 degrees
- moved C5 103.1 mm to (103.3, 65.1)
- moved C6 103.1 mm to (118.8, 67.6)
- moved C7 103.1 mm to (124.8, 64.6)
- moved D11 103.1 mm to (118.8, 36.1)
- moved MK1 103.1 mm to (101.0, 75.1)
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Routing:
- net Net-(D1-K): track 0.00 -> 203.4 mm, vias 0 -> 2
- net Net-(D8-A): track 0.00 -> 149.1 mm
- net Net-(D9-A): track 0.00 -> 109.7 mm
- net Net-(D10-A): track 0.00 -> 98.9 mm
- net Net-(D7-A): track 0.00 -> 69.1 mm, vias 0 -> 2
- net Net-(D5-A): track 0.00 -> 53.6 mm
- net Net-(D6-A): track 0.00 -> 46.8 mm, vias 0 -> 2
- net Net-(U4-THR): track 0.00 -> 43.8 mm
- net Net-(D4-A): track 0.00 -> 41.6 mm
- net Net-(U5-DIS): track 0.00 -> 32.9 mm, vias 0 -> 2
- net Net-(U1-DIS): track 0.00 -> 31.1 mm
- net Net-(U1-Q): track 0.00 -> 29.1 mm, vias 0 -> 2
- net Net-(U2A-+): track 0.00 -> 28.3 mm
- net Net-(D3-A): track 0.00 -> 22.6 mm
- net Net-(D11-A): track 0.00 -> 21.8 mm
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- added copper zone on B.Cu, net GND
Other:
- board size 182.8 x 90 mm -> 115 x 90 mm
- board text added: "C7"

Commit message: kicad updated
Other:
- board text added: "ANTONIA CRISTI NATALIA PILAR PAULINA VARGAS"
- board text added: "CIRCUITO RULETA"
- board text added: "G5"
- board text added: "MIC FALSO"
- board text added: "TALLER MAQUINAS ELECTRONICAS"
Changed lines of the file:
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@@
 		(tenting front back)
 		(pcbplotparams
-			(layerselection 0x00000000_00000000_55555555_575555f5)
+			(layerselection 0x00000000_00000000_55555555_575555ff)
 			(plot_on_all_layers_selection 0x00000000_00000000_00000000_00000000)
 			(disableapertmacros no)
@@
 			(drillshape 0)
 			(scaleselection 1)
-			(outputdirectory "C:/Users/napil/Downloads/taller/")
+			(outputdirectory "PCB 5G/")
 		)
 	)
@@
 		(layer "Edge.Cuts")
 	)
+	(gr_text "G5"
+		(at 46.26 45.24 0)
+		(layer "F.SilkS")
+		(effects
+			(font
+				(size 6 6)
+				(thickness 0.1)
+			)
+			(justify left bottom)
+		)
+	)
 	(gr_text "C7"
 		(at 124.75 62.5 0)
@@
 		)
 	)
+	(gr_text "CIRCUITO RULETA"
+		(at 57.18 113.295 0)
+		(layer "F.SilkS")
+		(effects
+			(font
+				(size 1.5 1.5)
+				(thickness 0.1)
+			)
+			(justify left bottom)
+		)
+	)
+	(gr_text "MIC FALSO"
+		(at 99.5 33 0)
+		(layer "F.SilkS")
+		(effects
+			(font
+				(size 1.5 1.5)
+				(thickness 0.1)
+			)
+			(justify left bottom)
+		)
+	)
+	(gr_text "TALLER\nMAQUINAS\nELECTRONICAS"
+		(at 126 80 0)
+		(layer "F.SilkS")
+		(effects
+			(font
+				(size 1.5 1.5)
+				(thickness 0.1)
+			)
+			(justify right bottom)
+		)
+	)
+	(gr_text "ANTONIA CRISTI\nNATALIA PILAR\nPAULINA VARGAS"
+		(at 77 45 0)
+		(layer "F.SilkS")
+		(effects
+			(font
+				(size 1.5 1.5)
+				(thickness 0.1)
+			)
+			(justify right bottom)
+		)
+	)
