File: 00-proyecto-02/grupo-06/kicad/fps555-kicad/fps555-v5.2.kicad_sch (KiCad schematic)
At the start: 23 parts, among them J1 Batería 9v, M1 Motorreductor, U1 555, U2 L293D, U3 mst303

Commit message: pcb
Other:
- moved on the sheet: C1, C2, D1, D2, D3, D4, D5, D6, D7, D8, J1, M1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
